File: kicad/bitamp/bitamp.kicad_sch (KiCad schematic)
At the start: 10 parts, among them J1 Jack-DC, J2 ToBitcaster, J3 ToPreamp, SW1 SW_SPST

Commit message: update kicad files
Parts:
- removed R3: R, symbol Device:R
- added D3: D_Schottky, symbol Device:D_Schottky
- C1: value 0.1uF -> 0.1µF; footprint (none) -> Capacitor_THT:C_Disc_D16.0mm_W5.0mm_P10.00mm
- D1: value PWR_LED -> LED_PWR; footprint (none) -> LED_THT:LED_D3.0mm_Clear
- D2: value BTC_LED -> LED_BTX; footprint (none) -> LED_THT:LED_D3.0mm_Clear
- J1: footprint (none) -> Connector_BarrelJack:BarrelJack_Horizontal
- J2, J3: footprint (none) -> Connector_Audio:Jack_6.35mm_Neutrik_NRJ6HM-1-PRE_Horizontal
- R1: value R -> 71.5Ω; footprint (none) -> Resistor_THT:R_Axial_Power_L20.0mm_W6.4mm_P5.08mm_Vertical
- R2: value R -> 210Ω; footprint (none) -> Resistor_THT:R_Axial_Power_L20.0mm_W6.4mm_P5.08mm_Vertical
- SW1: value SW_SPST -> SW_Stomp; footprint (none) -> Button_Switch_THT:SW_Push_1P1T_NO_LED_E-Switch_TL1250
Connections:
- net at J1.2, R1.1, R2.1: now also C1.2, D3.1 (K); no longer J2.R, J3.S
- net at D2.2 (A), SW1.2 (B): now also C1.1, J2.S; no longer C1.2
- new net: D3.2 (A), J2.R, J3.S
Other:
- moved on the sheet: C1, D1, D2, J1, J2, J3, R1, R2, SW1
